File: PCB_PracticeBoard/PCB_PracticeBoard.kicad_sch (KiCad schematic)
At the start: 31 parts, among them J1 UART0, J2 UART1, J3 I2C0, J4 I2C1, J5 Software_Serial, J6 Conn_01x03_Female, J7 18742, SW1 SW_Push, SW2 SW_Push, SW3 SW_DPDT_x2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

Commit message: create gerber files
Parts:
- C1: footprint LED_SMD:LED-APA102-2020 -> SamacSys_Parts:CAPPRD500W60D1025H1400
- C2, C3, C4, C5: footprint (none) -> SamacSys_Parts:CAPPRD500W60D1025H1400
- D1, D2, D3, D4: footprint (none) -> LED_THT:LED_D5.0mm
- J1, J2, J3, J4, J5: footprint (none) -> SamacSys_Parts:SHDRRA2W80P0X250_1X2_740X1150X610P
- J6: footprint (none) -> SamacSys_Parts:SHDRRA3W64P0X250_1X3_990X1150X610P
- J7: footprint 18742 -> SamacSys_Parts:18742
- R1, R2, R3, R4, R5, R6, R7, R8: footprint (none) -> Resistor_THT:R_Axial_DIN0207_L6.3mm_D2.5mm_P10.16mm_Horizontal
- RV1: footprint (none) -> SamacSys_Parts:3386K
- SW1, SW2, SW4, SW5: footprint (none) -> Button_Switch_THT:SW_PUSH_6mm_H4.3mm
- SW3: footprint (none) -> SamacSys_Parts:2MS1T2B4M2QES
- U1: footprint RPi_Pico:RPi_Pico_SMD_TH -> SamacSys_Parts:RPi_Pico_SMD_TH
Connections:
- net SW3: now also SW3.2 (B); no longer C4.1, R6.2
- net SW4: now also C4.1, R6.2; no longer C5.1, R8.2
- net SW5: now also C5.1, R8.2; no longer SW3.2 (B)
